File: eagle/sdmapper-jgilcas.sch (EAGLE design)
At the start: 27 parts, among them IC1 AM29F010E, IC2 HM628512ASOP32, IC3 XC95144XL_TQ100, IC4 LM1117-3V3, T1 BC858, T2 BC858, U1 USD-SOCKETUSD, X1 25MHz

Commit message: Add files via upload
Parts:
- removed D2: Cart2, led:LEDCHIP-LED0805
- removed R2: 4K7, rcl:R-EU_R0805
- removed T2: BC858, transistor:BC858A-PNP-SOT23-BEC
Connections:
- removed net N$5: R2.1, T2.B
- removed net N$9: D2.A, T2.C
- net +3V3: no longer T2.E
- net N$7: no longer D2.C
- net SD_CS1: no longer R2.2
